Commit message: Fixesfixesfixes

File: description/gazebo_control.xacro (robot description, xacro)
@@ -6,6 +6,6 @@
             <left_joint>left_wheel_joint</left_joint>
             <right_joint>right_wheel_joint</right_joint>
-            <wheel_separation>0.35</wheel_separation>
-            <wheel_diameter>0.1</wheel_diameter>
+            <wheel_separation>0.285</wheel_separation>
+            <wheel_diameter>0.099</wheel_diameter>
             <!-- Limits -->
             <max_wheel_torque>200</max_wheel_torque>

File: description/lidar.xacro (robot description, xacro)
@@ -2,7 +2,7 @@
 <robot xmlns:xacro="http://www.ros.org/wiki/xacro"  name="robot">
     <joint name="laser_joint" type="fixed">
-        <parent link="chassis"/>
+        <parent link="wheelbase"/>
         <child link="laser_frame"/>
-        <origin xyz="0.1 0 0.175" rpy="0 0 0"/>
+        <origin xyz="0 0 0.09561" rpy="0 0 0"/>
     </joint>
     <link name="laser_frame">
@@ -45,5 +45,5 @@
                     <argument>~/out:=scan</argument>
                 </ros>
-                <output_type>sensor_msgs/LaserScam</output_type>
+                <output_type>sensor_msgs/LaserScan</output_type>
                 <frame_name>laser_frame</frame_name>
             </plugin>

File: description/robot_core.xacro (robot description, xacro)
@@ -19,26 +19,53 @@
     <link name="base_link">
     </link>
+   <!-- Wheelbase -->
+    <joint name="wheelbase_joint" type="fixed">
+        <parent link="base_link"/>
+        <child link="wheelbase"/>
+        <origin xyz="0 0 0.0121"/>
+    </joint>
+    <link name="wheelbase">
+        <visual>
+            <origin xyz="0 0 0" rpy="0 0 0"/>
+            <geometry>
+                <box size="0.075 0.24 0.046"/>
+            </geometry>
+            <material name="black"/>
+        </visual>
+        <collision>
+            <origin xyz="0 0 0" rpy="0 0 0"/>
+            <geometry>
+                <box size="0.075 0.24 0.046"/>
+            </geometry>
+        </collision>
+        <xacro:inertial_box mass="0.5" x="0.075" y="0.24" z="0.046">
+            <origin xyz="0 0 0" rpy="0 0 0"/>
+        </xacro:inertial_box>
+    </link>
+    <gazebo reference="wheelbase">
+        <material>Gazebo/Black</material>
+    </gazebo>
     <!-- CHASSIS -->
     <joint name="chassis_joint" type="fixed">
-        <parent link="base_link"/>
+        <parent link="wheelbase"/>
         <child link="chassis"/>
-        <origin xyz="-0.1 0 0"/>
+        <origin xyz="-0.0725 0 0.02685"/>
     </joint>
     <link name="chassis">
         <visual>
-            <origin xyz="0.15 0 0.075" rpy="0 0 0"/>
+            <origin xyz="0 0 0" rpy="0 0 0"/>
             <geometry>
-                <box size="0.3 0.3 0.15"/>
+                <box size="0.33 0.24 0.0077"/>
             </geometry>
             <material name="orange"/>
         </visual>
         <collision>
-            <origin xyz="0.15 0 0.075" rpy="0 0 0"/>
+            <origin xyz="0 0 0" rpy="0 0 0"/>
             <geometry>
-                <box size="0.3 0.3 0.15"/>
+                <box size="0.33 0.24 0.0077"/>
             </geometry>
         </collision>
-        <xacro:inertial_box mass="0.5" x="0.3" y="0.3" z="0.15">
-            <origin xyz="0.15 0 0.075" rpy="0 0 0"/>
+        <xacro:inertial_box mass="1.027" x="0.33" y="0.24" z="0.0077">
+            <origin xyz="0 0 0" rpy="0 0 0"/>
         </xacro:inertial_box>
     </link>
@@ -50,5 +77,5 @@
         <parent link="base_link"/>
         <child link="right_wheel"/>
-        <origin xyz="0 -0.175 0" rpy="${pi/2} 0 0"/>
+        <origin xyz="0 -0.1425 0" rpy="${pi/2} 0 0"/>
         <axis xyz="0 0 -1"/>
     </joint>
@@ -57,56 +84,57 @@
             <origin xyz="0 0 0" rpy="0 0 0"/>
             <geometry>
-                <cylinder length="0.04" radius="0.05" />
+                <cylinder length="0.0265" radius="0.0495" />
             </geometry>
-        <material name="blue"/>
+        <material name="white"/>
         </visual>
         <collision>
             <geometry>
-                <cylinder length="0.04" radius="0.05" />
+                <cylinder length="0.0265" radius="0.0495" />
             </geometry>
         </collision>
-        <xacro:inertial_cylinder mass="0.1" length="0.05" radius="0.05">
+        <xacro:inertial_cylinder mass="0.134" length="0.0265" radius="0.0495">
             <origin xyz="0 0 0" rpy="0 0 0"/>
         </xacro:inertial_cylinder>
     </link>
     <gazebo reference="right_wheel">
-        <material>Gazebo/Blue</material>
+        <material>Gazebo/White</material>
     </gazebo>
 	<!-- LEFT WHEEL -->
-	<joint name="left_wheel_joint" type="continuous">
-	    <parent link="base_link"/>
-	    <child link="left_wheel"/>
-	    <origin xyz="0 0.175 0" rpy="-${pi/2} 0 0"/>
-	    <axis xyz="0 0 1"/>
-	</joint>
-	<link name="left_wheel">
-	    <visual>
+    <joint name="left_wheel_joint" type="continuous">
+        <parent link="base_link"/>
+        <child link="left_wheel"/>
+        <origin xyz="0 0.1425 0" rpy="${pi/2} 0 0"/>
+        <axis xyz="0 0 -1"/>
+    </joint>
+    <link name="left_wheel">
+        <visual>
+            <origin xyz="0 0 0" rpy="0 0 0"/>
             <geometry>
-                <cylinder length="0.04" radius="0.05" />
+                <cylinder length="0.0265" radius="0.0495" />
             </geometry>
-		    <material name="blue"/>
-	    </visual>
+        <material name="white"/>
+        </visual>
         <collision>
             <geometry>
-                <cylinder length="0.04" radius="0.05" />
+                <cylinder length="0.0265" radius="0.0495" />
             </geometry>
         </collision>
-        <xacro:inertial_cylinder mass="0.1" length="0.05" radius="0.05">
+        <xacro:inertial_cylinder mass="0.134" length="0.0265" radius="0.0495">
             <origin xyz="0 0 0" rpy="0 0 0"/>
         </xacro:inertial_cylinder>
-	</link>
+    </link>
     <gazebo reference="left_wheel">
-        <material>Gazebo/Blue</material>
+        <material>Gazebo/White</material>
     </gazebo>
     <!-- CASTER WHEEL -->
     <joint name="caster_wheel_joint" type="fixed">
-        <parent link="chassis"/>
+        <parent link="base_link"/>
         <child link="caster_wheel"/>
-        <origin xyz="0.24 0 0" rpy="0 0 0"/>
+        <origin xyz="-0.18 0 0" rpy="0 0 0"/>
     </joint>
     <link name="caster_wheel">
         <visual>
             <geometry>
-                <sphere radius="0.05" />
+                <sphere radius="0.0495" />
             </geometry>
             <material name="black"/>
@@ -114,8 +142,8 @@
         <collision>
             <geometry>
-                <sphere radius="0.05" />
+                <sphere radius="0.0495" />
             </geometry>
         </collision>
-        <xacro:inertial_sphere mass="0.1" radius="0.05">
+        <xacro:inertial_sphere mass="0.2" radius="0.0495">
             <origin xyz="0 0 0" rpy="0 0 0"/>
         </xacro:inertial_sphere>
