Commit message: robot description fix

File: description/camera.xacro (robot description, xacro)
@@ -4,5 +4,5 @@
         <parent link="wheelbase"/>
         <child link="camera_link"/>
-        <origin xyz="0.0925 0 0.0457" rpy="0 0 0"/>
+        <origin xyz="-0.09 0 0.0457" rpy="0 0 0"/>
     </joint>
     <link name="camera_link">

File: description/robot_core.xacro (robot description, xacro)
@@ -105,5 +105,5 @@
         <child link="left_wheel"/>
         <origin xyz="0 0.1425 0" rpy="${pi/2} 0 0"/>
-        <axis xyz="0 0 -1"/>
+        <axis xyz="0 0 1"/>
     </joint>
     <link name="left_wheel">

Commit message: foxed camera position

File: description/camera.xacro (robot description, xacro)
@@ -4,5 +4,5 @@
         <parent link="wheelbase"/>
         <child link="camera_link"/>
-        <origin xyz="-0.09 0 0.0457" rpy="0 0 0"/>
+        <origin xyz="0.09 0 0.0457" rpy="0 0 0"/>
     </joint>
     <link name="camera_link">

Commit message: fixed camera and lidar positions

File: description/camera.xacro (robot description, xacro)
@@ -4,5 +4,5 @@
         <parent link="wheelbase"/>
         <child link="camera_link"/>
-        <origin xyz="0.0925 0 0.0457" rpy="0 0 0"/>
+        <origin xyz="0.0925 0 0.0687" rpy="0 0 0"/>
     </joint>
     <link name="camera_link">

File: description/lidar.xacro (robot description, xacro)
@@ -4,5 +4,5 @@
         <parent link="wheelbase"/>
         <child link="laser_frame"/>
-        <origin xyz="0 0 0.09561" rpy="0 0 0"/>
+        <origin xyz="0 0 0.11061" rpy="0 0 0"/>
     </joint>
     <link name="laser_frame">
