Commit message: fixed wheel joints

File: description/robot_core.xacro (robot description, xacro)
@@ -74,5 +74,5 @@
     </gazebo>
     <!-- RIGHT WHEEL -->
-    <joint name="right_wheel_joint" type="continuous">
+    <joint name="right_wheel_joint" type="revolute">
         <parent link="base_link"/>
         <child link="right_wheel"/>
@@ -101,5 +101,5 @@
     </gazebo>
 	<!-- LEFT WHEEL -->
-    <joint name="left_wheel_joint" type="continuous">
+    <joint name="left_wheel_joint" type="revolute">
         <parent link="base_link"/>
         <child link="left_wheel"/>

Commit message: fixed wheel joints

File: description/robot_core.xacro (robot description, xacro)
@@ -74,5 +74,5 @@
     </gazebo>
     <!-- RIGHT WHEEL -->
-    <joint name="right_wheel_joint" type="revolute">
+    <joint name="right_wheel_joint" type="continuous">
         <parent link="base_link"/>
         <child link="right_wheel"/>
@@ -101,5 +101,5 @@
     </gazebo>
 	<!-- LEFT WHEEL -->
-    <joint name="left_wheel_joint" type="revolute">
+    <joint name="left_wheel_joint" type="continuous">
         <parent link="base_link"/>
         <child link="left_wheel"/>
